File: 12ax7_socket/12ax7_socket.kicad_sch (KiCad schematic)
At the start: 2 parts, among them J1 Conn_01x09, U1 ECC83

Commit message: Fix footprint of valve socket
Parts:
- U1: footprint tube_breakouts:Valve_12AX7_Socket -> kosmo-lib:Valve_12AX7_Socket
Changed lines of the file:
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@@
       (effects (font (size 1.27 1.27)) (justify left))
     )
-    (property "Footprint" "tube_breakouts:Valve_12AX7_Socket" (id 2) (at 95.758 99.06 0)
+    (property "Footprint" "kosmo-lib:Valve_12AX7_Socket" (id 2) (at 95.758 99.06 0)
       (effects (font (size 1.27 1.27)) hide)
     )
@@
       (effects (font (size 1.27 1.27)) (justify left))
     )
-    (property "Footprint" "tube_breakouts:Valve_12AX7_Socket" (id 2) (at 171.958 99.06 0)
+    (property "Footprint" "kosmo-lib:Valve_12AX7_Socket" (id 2) (at 171.958 99.06 0)
       (effects (font (size 1.27 1.27)) hide)
     )
@@
       (effects (font (size 1.27 1.27)) (justify left))
     )
-    (property "Footprint" "tube_breakouts:Valve_12AX7_Socket" (id 2) (at 133.858 99.06 0)
+    (property "Footprint" "kosmo-lib:Valve_12AX7_Socket" (id 2) (at 133.858 99.06 0)
       (effects (font (size 1.27 1.27)) hide)
     )
@@
     )
     (path "/b99f1e04-ee9c-4ddc-bec0-6bfa50d749dc"
-      (reference "U1") (unit 1) (value "ECC83") (footprint "tube_breakouts:Valve_12AX7_Socket")
+      (reference "U1") (unit 1) (value "ECC83") (footprint "kosmo-lib:Valve_12AX7_Socket")
     )
     (path "/3b748e42-cf71-4ebf-86b0-2d022229e4b6"
-      (reference "U1") (unit 2) (value "ECC83") (footprint "tube_breakouts:Valve_12AX7_Socket")
+      (reference "U1") (unit 2) (value "ECC83") (footprint "kosmo-lib:Valve_12AX7_Socket")
     )
     (path "/8685b77e-a02f-4ac0-b515-6aad8ce186bf"
-      (reference "U1") (unit 3) (value "ECC83") (footprint "tube_breakouts:Valve_12AX7_Socket")
+      (reference "U1") (unit 3) (value "ECC83") (footprint "kosmo-lib:Valve_12AX7_Socket")
     )
   )
